File: PortA.sch (KiCad schematic (older format))
At the start: 1 part, among them U3 XC7010-1CLG400C_AzizFaozi

Commit message: add some pmic library
Parts:
- U3: symbol MedusaLIB:XC7010-1CLG400C_AzizFaozi -> MedusaSDR-rescue:XC7010-1CLG400C_AzizFaozi-MedusaLIB
Changed lines of the file:
@@
 EESchema Schematic File Version 4
-LIBS:MedusaSDR-cache
 EELAYER 30 0
 EELAYER END
 $Descr A3 16535 11693
 encoding utf-8
-Sheet 4 11
+Sheet 4 12
 Title ""
 Date ""
@@
 $EndDescr
 $Comp
-L MedusaLIB:XC7010-1CLG400C_AzizFaozi U3
+L MedusaSDR-rescue:XC7010-1CLG400C_AzizFaozi-MedusaLIB U3
 U 5 1 5DE66979
 P 4150 3100
@@
 $EndComp
 $Comp
-L MedusaLIB:XC7010-1CLG400C_AzizFaozi U3
+L MedusaSDR-rescue:XC7010-1CLG400C_AzizFaozi-MedusaLIB U3
 U 6 1 5DE673FF
 P 11850 3600
@@
 $EndComp
 $Comp
-L MedusaLIB:XC7010-1CLG400C_AzizFaozi U3
+L MedusaSDR-rescue:XC7010-1CLG400C_AzizFaozi-MedusaLIB U3
 U 7 1 5DE78BB8
 P 4000 8050
@@
 $EndComp
 $Comp
-L MedusaLIB:XC7010-1CLG400C_AzizFaozi U3
+L MedusaSDR-rescue:XC7010-1CLG400C_AzizFaozi-MedusaLIB U3
 U 8 1 5DE85FA7
 P 11900 8200
@@
 	10450 3700 11100 3700
 $Comp
-L power:GND #PWR?
+L power:GND #PWR02
 U 1 1 5DFAFBC4
 P 3000 8450
-F 0 "#PWR?" H 3000 8200 50  0001 C CNN
+F 0 "#PWR02" H 3000 8200 50  0001 C CNN
 F 1 "GND" V 3005 8322 50  0000 R CNN
 F 2 "" H 3000 8450 50  0001 C CNN
@@
 	3000 8450 3250 8450
 $Comp
-L power:GND #PWR?
+L power:GND #PWR04
 U 1 1 5DFB2472
 P 4950 8350
-F 0 "#PWR?" H 4950 8100 50  0001 C CNN
+F 0 "#PWR04" H 4950 8100 50  0001 C CNN
 F 1 "GND" V 4955 8222 50  0000 R CNN
 F 2 "" H 4950 8350 50  0001 C CNN
@@
 	4700 8350 4950 8350
 $Comp
-L power:GND #PWR?
+L power:GND #PWR03
 U 1 1 5DFB69B9
 P 4950 7950
-F 0 "#PWR?" H 4950 7700 50  0001 C CNN
+F 0 "#PWR03" H 4950 7700 50  0001 C CNN
 F 1 "GND" V 4955 7822 50  0000 R CNN
 F 2 "" H 4950 7950 50  0001 C CNN
