File: PortB.sch (KiCad schematic (older format))
At the start: 1 part, among them U3 XC7010-1CLG400C_AzizFaozi

Commit message: add some pmic library
Parts:
- U3: symbol MedusaLIB:XC7010-1CLG400C_AzizFaozi -> MedusaSDR-rescue:XC7010-1CLG400C_AzizFaozi-MedusaLIB
Changed lines of the file:
@@
 EESchema Schematic File Version 4
-LIBS:MedusaSDR-cache
 EELAYER 30 0
 EELAYER END
 $Descr A3 16535 11693
 encoding utf-8
-Sheet 3 11
+Sheet 3 12
 Title ""
 Date ""
@@
 $EndDescr
 $Comp
-L MedusaLIB:XC7010-1CLG400C_AzizFaozi U3
+L MedusaSDR-rescue:XC7010-1CLG400C_AzizFaozi-MedusaLIB U3
 U 2 1 5DDDDC60
 P 12700 3100
@@
 $EndComp
 $Comp
-L MedusaLIB:XC7010-1CLG400C_AzizFaozi U3
+L MedusaSDR-rescue:XC7010-1CLG400C_AzizFaozi-MedusaLIB U3
 U 1 1 5DDD2E26
 P 4250 2800
@@
 	14050 3500 14050 3550
 $Comp
-L MedusaLIB:XC7010-1CLG400C_AzizFaozi U3
+L MedusaSDR-rescue:XC7010-1CLG400C_AzizFaozi-MedusaLIB U3
 U 3 1 5DE4552A
 P 4550 8000
@@
 $EndComp
 $Comp
-L MedusaLIB:XC7010-1CLG400C_AzizFaozi U3
+L MedusaSDR-rescue:XC7010-1CLG400C_AzizFaozi-MedusaLIB U3
 U 4 1 5DE58A35
 P 12150 7850
@@
 $EndComp
 $Comp
-L power:GND #PWR?
+L power:GND #PWR01
 U 1 1 5E036625
 P 3300 8300
-F 0 "#PWR?" H 3300 8050 50  0001 C CNN
+F 0 "#PWR01" H 3300 8050 50  0001 C CNN
 F 1 "GND" V 3305 8172 50  0000 R CNN
 F 2 "" H 3300 8300 50  0001 C CNN
