File: PortC.sch (KiCad schematic (older format))
At the start: 1 part, among them U3 XC7010-1CLG400C_AzizFaozi

Commit message: add some pmic library
Parts:
- U3: symbol MedusaLIB:XC7010-1CLG400C_AzizFaozi -> MedusaSDR-rescue:XC7010-1CLG400C_AzizFaozi-MedusaLIB
Changed lines of the file:
@@
 EESchema Schematic File Version 4
-LIBS:MedusaSDR-cache
 EELAYER 30 0
 EELAYER END
 $Descr A3 16535 11693
 encoding utf-8
-Sheet 5 11
+Sheet 5 12
 Title ""
 Date ""
@@
 $EndDescr
 $Comp
-L MedusaLIB:XC7010-1CLG400C_AzizFaozi U3
+L MedusaSDR-rescue:XC7010-1CLG400C_AzizFaozi-MedusaLIB U3
 U 9 1 5DEEB517
 P 4350 2700
@@
 $EndComp
 $Comp
-L MedusaLIB:XC7010-1CLG400C_AzizFaozi U3
+L MedusaSDR-rescue:XC7010-1CLG400C_AzizFaozi-MedusaLIB U3
 U 10 1 5DEEC31A
 P 12550 3200
@@
 $EndComp
 $Comp
-L MedusaLIB:XC7010-1CLG400C_AzizFaozi U3
+L MedusaSDR-rescue:XC7010-1CLG400C_AzizFaozi-MedusaLIB U3
 U 11 1 5DEF435C
 P 4200 7650
@@
 $EndComp
 $Comp
-L MedusaLIB:XC7010-1CLG400C_AzizFaozi U3
+L MedusaSDR-rescue:XC7010-1CLG400C_AzizFaozi-MedusaLIB U3
 U 12 1 5DEF61CE
 P 12550 8000
@@
 	4900 7850 5250 7850
 $Comp
-L power:GND #PWR?
+L power:GND #PWR05
 U 1 1 5E0091E2
 P 3300 2700
-F 0 "#PWR?" H 3300 2450 50  0001 C CNN
+F 0 "#PWR05" H 3300 2450 50  0001 C CNN
 F 1 "GND" V 3305 2572 50  0000 R CNN
 F 2 "" H 3300 2700 50  0001 C CNN
@@
 $EndComp
 $Comp
-L power:GND #PWR?
+L power:GND #PWR07
 U 1 1 5E00A7A9
 P 5300 2600
-F 0 "#PWR?" H 5300 2350 50  0001 C CNN
+F 0 "#PWR07" H 5300 2350 50  0001 C CNN
 F 1 "GND" V 5305 2472 50  0000 R CNN
 F 2 "" H 5300 2600 50  0001 C CNN
@@
 	5050 2600 5300 2600
 $Comp
-L power:GND #PWR?
+L power:GND #PWR06
 U 1 1 5E011EB4
 P 5250 8050
-F 0 "#PWR?" H 5250 7800 50  0001 C CNN
+F 0 "#PWR06" H 5250 7800 50  0001 C CNN
 F 1 "GND" V 5255 7922 50  0000 R CNN
 F 2 "" H 5250 8050 50  0001 C CNN
