File: PortD.sch (KiCad schematic (older format))
At the start: 4 parts

Commit message: add some pmic library
Parts:
- U3: renamed from U?; symbol MedusaLIB:XC7010-1CLG400C_AzizFaozi -> MedusaSDR-rescue:XC7010-1CLG400C_AzizFaozi-MedusaLIB
Changed lines of the file:
@@
 EESchema Schematic File Version 4
-LIBS:MedusaSDR-cache
 EELAYER 30 0
 EELAYER END
 $Descr A3 16535 11693
 encoding utf-8
-Sheet 6 11
+Sheet 6 12
 Title ""
 Date ""
@@
 $EndDescr
 $Comp
-L MedusaLIB:XC7010-1CLG400C_AzizFaozi U?
+L MedusaSDR-rescue:XC7010-1CLG400C_AzizFaozi-MedusaLIB U3
 U 13 1 5DF3B46D
 P 4150 3100
-F 0 "U?" H 4125 3865 50  0000 C CNN
+F 0 "U3" H 4125 3865 50  0000 C CNN
 F 1 "XC7010-1CLG400C_AzizFaozi" H 4125 3774 50  0000 C CNN
 F 2 "Package_BGA:Xilinx_CLG400" H 4100 2450 50  0001 C CNN
@@
 $EndComp
 $Comp
-L MedusaLIB:XC7010-1CLG400C_AzizFaozi U?
+L MedusaSDR-rescue:XC7010-1CLG400C_AzizFaozi-MedusaLIB U3
 U 14 1 5DF4DF7A
 P 12150 3150
-F 0 "U?" H 12125 3915 50  0000 C CNN
+F 0 "U3" H 12125 3915 50  0000 C CNN
 F 1 "XC7010-1CLG400C_AzizFaozi" H 12125 3824 50  0000 C CNN
 F 2 "Package_BGA:Xilinx_CLG400" H 12100 2500 50  0001 C CNN
@@
 $EndComp
 $Comp
-L MedusaLIB:XC7010-1CLG400C_AzizFaozi U?
+L MedusaSDR-rescue:XC7010-1CLG400C_AzizFaozi-MedusaLIB U3
 U 15 1 5DF5B016
 P 4100 7400
-F 0 "U?" H 4075 8165 50  0000 C CNN
+F 0 "U3" H 4075 8165 50  0000 C CNN
 F 1 "XC7010-1CLG400C_AzizFaozi" H 4075 8074 50  0000 C CNN
 F 2 "Package_BGA:Xilinx_CLG400" H 4050 6750 50  0001 C CNN
@@
 $EndComp
 $Comp
-L MedusaLIB:XC7010-1CLG400C_AzizFaozi U?
+L MedusaSDR-rescue:XC7010-1CLG400C_AzizFaozi-MedusaLIB U3
 U 16 1 5DF6768B
 P 12250 7150
-F 0 "U?" H 12225 7915 50  0000 C CNN
+F 0 "U3" H 12225 7915 50  0000 C CNN
 F 1 "XC7010-1CLG400C_AzizFaozi" H 12225 7824 50  0000 C CNN
 F 2 "Package_BGA:Xilinx_CLG400" H 12200 6500 50  0001 C CNN
@@
 $EndComp
 $Comp
-L power:GND #PWR?
+L power:GND #PWR09
 U 1 1 5DFBB05B
 P 3150 2600
-F 0 "#PWR?" H 3150 2350 50  0001 C CNN
+F 0 "#PWR09" H 3150 2350 50  0001 C CNN
 F 1 "GND" V 3155 2472 50  0000 R CNN
 F 2 "" H 3150 2600 50  0001 C CNN
@@
 $EndComp
 $Comp
-L power:GND #PWR?
+L power:GND #PWR010
 U 1 1 5DFBC304
 P 3150 3200
-F 0 "#PWR?" H 3150 2950 50  0001 C CNN
+F 0 "#PWR010" H 3150 2950 50  0001 C CNN
 F 1 "GND" V 3155 3072 50  0000 R CNN
 F 2 "" H 3150 3200 50  0001 C CNN
@@
 $EndComp
 $Comp
-L power:GND #PWR?
+L power:GND #PWR012
 U 1 1 5DFBD642
 P 5050 3500
-F 0 "#PWR?" H 5050 3250 50  0001 C CNN
+F 0 "#PWR012" H 5050 3250 50  0001 C CNN
 F 1 "GND" V 5055 3372 50  0000 R CNN
 F 2 "" H 5050 3500 50  0001 C CNN
@@
 $EndComp
 $Comp
-L power:GND #PWR?
+L power:GND #PWR011
 U 1 1 5DFBE9C5
 P 5050 3300
-F 0 "#PWR?" H 5050 3050 50  0001 C CNN
+F 0 "#PWR011" H 5050 3050 50  0001 C CNN
 F 1 "GND" V 5055 3172 50  0000 R CNN
 F 2 "" H 5050 3300 50  0001 C CNN
@@
 	3150 2600 3400 2600
 $Comp
-L power:GND #PWR?
+L power:GND #PWR016
 U 1 1 5DFC6431
 P 11100 2950
-F 0 "#PWR?" H 11100 2700 50  0001 C CNN
+F 0 "#PWR016" H 11100 2700 50  0001 C CNN
 F 1 "GND" V 11105 2822 50  0000 R CNN
 F 2 "" H 11100 2950 50  0001 C CNN
@@
 $EndComp
 $Comp
-L power:GND #PWR?
+L power:GND #PWR017
 U 1 1 5DFC783A
 P 11100 3350
-F 0 "#PWR?" H 11100 3100 50  0001 C CNN
+F 0 "#PWR017" H 11100 3100 50  0001 C CNN
 F 1 "GND" V 11105 3222 50  0000 R CNN
 F 2 "" H 11100 3350 50  0001 C CNN
@@
 $EndComp
 $Comp
-L power:GND #PWR?
+L power:GND #PWR018
 U 1 1 5DFC8C26
 P 11100 3550
-F 0 "#PWR?" H 11100 3300 50  0001 C CNN
+F 0 "#PWR018" H 11100 3300 50  0001 C CNN
 F 1 "GND" V 11105 3422 50  0000 R CNN
 F 2 "" H 11100 3550 50  0001 C CNN
@@
 $EndComp
 $Comp
-L power:GND #PWR?
+L power:GND #PWR020
 U 1 1 5DFCAC5A
 P 13150 3450
-F 0 "#PWR?" H 13150 3200 50  0001 C CNN
+F 0 "#PWR020" H 13150 3200 50  0001 C CNN
 F 1 "GND" V 13155 3322 50  0000 R CNN
 F 2 "" H 13150 3450 50  0001 C CNN
@@
 $EndComp
 $Comp
-L power:GND #PWR?
+L power:GND #PWR019
 U 1 1 5DFCB1F4
 P 13150 3250
-F 0 "#PWR?" H 13150 3000 50  0001 C CNN
+F 0 "#PWR019" H 13150 3000 50  0001 C CNN
 F 1 "GND" V 13155 3122 50  0000 R CNN
 F 2 "" H 13150 3250 50  0001 C CNN
@@
 	11100 2950 11400 2950
 $Comp
-L power:GND #PWR?
+L power:GND #PWR014
 U 1 1 5DFD1ED2
 P 11050 7250
-F 0 "#PWR?" H 11050 7000 50  0001 C CNN
+F 0 "#PWR014" H 11050 7000 50  0001 C CNN
 F 1 "GND" V 11055 7122 50  0000 R CNN
 F 2 "" H 11050 7250 50  0001 C CNN
@@
 	11050 7250 11500 7250
 $Comp
-L power:GND #PWR?
+L power:GND #PWR015
 U 1 1 5DFD46CF
 P 11050 7450
-F 0 "#PWR?" H 11050 7200 50  0001 C CNN
+F 0 "#PWR015" H 11050 7200 50  0001 C CNN
 F 1 "GND" V 11055 7322 50  0000 R CNN
 F 2 "" H 11050 7450 50  0001 C CNN
@@
 	11050 7450 11500 7450
 $Comp
-L power:GND #PWR?
+L power:GND #PWR021
 U 1 1 5DFD6D78
 P 13300 7550
-F 0 "#PWR?" H 13300 7300 50  0001 C CNN
+F 0 "#PWR021" H 13300 7300 50  0001 C CNN
 F 1 "GND" V 13305 7422 50  0000 R CNN
 F 2 "" H 13300 7550 50  0001 C CNN
@@
 	13300 7550 12950 7550
 $Comp
-L power:GND #PWR?
+L power:GND #PWR023
 U 1 1 5DFD93FB
 P 13350 7350
-F 0 "#PWR?" H 13350 7100 50  0001 C CNN
+F 0 "#PWR023" H 13350 7100 50  0001 C CNN
 F 1 "GND" V 13355 7222 50  0000 R CNN
 F 2 "" H 13350 7350 50  0001 C CNN
@@
 	13350 7350 12950 7350
 $Comp
-L power:GND #PWR?
+L power:GND #PWR022
 U 1 1 5DFDB90D
 P 13350 6950
-F 0 "#PWR?" H 13350 6700 50  0001 C CNN
+F 0 "#PWR022" H 13350 6700 50  0001 C CNN
 F 1 "GND" V 13355 6822 50  0000 R CNN
 F 2 "" H 13350 6950 50  0001 C CNN
@@
 	12950 6950 13350 6950
 $Comp
-L power:GND #PWR?
+L power:GND #PWR08
 U 1 1 5DFE1F1D
 P 2950 7700
-F 0 "#PWR?" H 2950 7450 50  0001 C CNN
+F 0 "#PWR08" H 2950 7450 50  0001 C CNN
 F 1 "GND" V 2955 7572 50  0000 R CNN
 F 2 "" H 2950 7700 50  0001 C CNN
@@
 	2950 7700 3350 7700
 $Comp
-L power:GND #PWR?
+L power:GND #PWR013
 U 1 1 5DFE37AC
 P 5250 7000
-F 0 "#PWR?" H 5250 6750 50  0001 C CNN
+F 0 "#PWR013" H 5250 6750 50  0001 C CNN
 F 1 "GND" V 5255 6872 50  0000 R CNN
 F 2 "" H 5250 7000 50  0001 C CNN
