File: PortE.sch (KiCad schematic (older format))
At the start: 4 parts

Commit message: add some pmic library
Parts:
- U3: renamed from U?; symbol MedusaLIB:XC7010-1CLG400C_AzizFaozi -> MedusaSDR-rescue:XC7010-1CLG400C_AzizFaozi-MedusaLIB
Changed lines of the file:
@@
 EESchema Schematic File Version 4
-LIBS:MedusaSDR-cache
 EELAYER 30 0
 EELAYER END
 $Descr A3 16535 11693
 encoding utf-8
-Sheet 7 11
+Sheet 7 12
 Title ""
 Date ""
@@
 $EndDescr
 $Comp
-L MedusaLIB:XC7010-1CLG400C_AzizFaozi U?
+L MedusaSDR-rescue:XC7010-1CLG400C_AzizFaozi-MedusaLIB U3
 U 17 1 5DF722E3
 P 3350 2350
-F 0 "U?" H 3325 3115 50  0000 C CNN
+F 0 "U3" H 3325 3115 50  0000 C CNN
 F 1 "XC7010-1CLG400C_AzizFaozi" H 3325 3024 50  0000 C CNN
 F 2 "Package_BGA:Xilinx_CLG400" H 3300 1700 50  0001 C CNN
@@
 $EndComp
 $Comp
-L MedusaLIB:XC7010-1CLG400C_AzizFaozi U?
+L MedusaSDR-rescue:XC7010-1CLG400C_AzizFaozi-MedusaLIB U3
 U 18 1 5DF84113
 P 11800 2300
-F 0 "U?" H 11775 3065 50  0000 C CNN
+F 0 "U3" H 11775 3065 50  0000 C CNN
 F 1 "XC7010-1CLG400C_AzizFaozi" H 11775 2974 50  0000 C CNN
 F 2 "Package_BGA:Xilinx_CLG400" H 11750 1650 50  0001 C CNN
@@
 $EndComp
 $Comp
-L MedusaLIB:XC7010-1CLG400C_AzizFaozi U?
+L MedusaSDR-rescue:XC7010-1CLG400C_AzizFaozi-MedusaLIB U3
 U 19 1 5DF8A9CF
 P 5550 6450
-F 0 "U?" H 5525 7215 50  0000 C CNN
+F 0 "U3" H 5525 7215 50  0000 C CNN
 F 1 "XC7010-1CLG400C_AzizFaozi" H 5525 7124 50  0000 C CNN
 F 2 "Package_BGA:Xilinx_CLG400" H 5500 5800 50  0001 C CNN
@@
 $EndComp
 $Comp
-L MedusaLIB:XC7010-1CLG400C_AzizFaozi U?
+L MedusaSDR-rescue:XC7010-1CLG400C_AzizFaozi-MedusaLIB U3
 U 20 1 5DF92692
 P 11600 6800
-F 0 "U?" H 11575 7565 50  0000 C CNN
+F 0 "U3" H 11575 7565 50  0000 C CNN
 F 1 "XC7010-1CLG400C_AzizFaozi" H 11575 7474 50  0000 C CNN
 F 2 "Package_BGA:Xilinx_CLG400" H 11550 6150 50  0001 C CNN
@@
 $EndComp
 $Comp
-L power:GND #PWR?
+L power:GND #PWR030
 U 1 1 5DFE78CF
 P 10550 2500
-F 0 "#PWR?" H 10550 2250 50  0001 C CNN
+F 0 "#PWR030" H 10550 2250 50  0001 C CNN
 F 1 "GND" V 10555 2372 50  0000 R CNN
 F 2 "" H 10550 2500 50  0001 C CNN
@@
 	11050 2500 10550 2500
 $Comp
-L power:GND #PWR?
+L power:GND #PWR033
 U 1 1 5DFE9ED2
 P 12850 2600
-F 0 "#PWR?" H 12850 2350 50  0001 C CNN
+F 0 "#PWR033" H 12850 2350 50  0001 C CNN
 F 1 "GND" V 12855 2472 50  0000 R CNN
 F 2 "" H 12850 2600 50  0001 C CNN
@@
 	12500 2600 12850 2600
 $Comp
-L power:GND #PWR?
+L power:GND #PWR032
 U 1 1 5DFEC2C0
 P 12850 1800
-F 0 "#PWR?" H 12850 1550 50  0001 C CNN
+F 0 "#PWR032" H 12850 1550 50  0001 C CNN
 F 1 "GND" V 12855 1672 50  0000 R CNN
 F 2 "" H 12850 1800 50  0001 C CNN
@@
 	12500 1800 12850 1800
 $Comp
-L power:GND #PWR?
+L power:GND #PWR028
 U 1 1 5DFF0777
 P 10500 6500
-F 0 "#PWR?" H 10500 6250 50  0001 C CNN
+F 0 "#PWR028" H 10500 6250 50  0001 C CNN
 F 1 "GND" V 10505 6372 50  0000 R CNN
 F 2 "" H 10500 6500 50  0001 C CNN
@@
 $EndComp
 $Comp
-L power:GND #PWR?
+L power:GND #PWR029
 U 1 1 5DFF183A
 P 10500 6900
-F 0 "#PWR?" H 10500 6650 50  0001 C CNN
+F 0 "#PWR029" H 10500 6650 50  0001 C CNN
 F 1 "GND" V 10505 6772 50  0000 R CNN
 F 2 "" H 10500 6900 50  0001 C CNN
@@
 $EndComp
 $Comp
-L power:GND #PWR?
+L power:GND #PWR031
 U 1 1 5DFF2C17
 P 12550 7000
-F 0 "#PWR?" H 12550 6750 50  0001 C CNN
+F 0 "#PWR031" H 12550 6750 50  0001 C CNN
 F 1 "GND" V 12555 6872 50  0000 R CNN
 F 2 "" H 12550 7000 50  0001 C CNN
@@
 	12300 7000 12550 7000
 $Comp
-L power:GND #PWR?
+L power:GND #PWR026
 U 1 1 5DFF7C85
 P 4500 6350
-F 0 "#PWR?" H 4500 6100 50  0001 C CNN
+F 0 "#PWR026" H 4500 6100 50  0001 C CNN
 F 1 "GND" V 4505 6222 50  0000 R CNN
 F 2 "" H 4500 6350 50  0001 C CNN
@@
 $EndComp
 $Comp
-L power:GND #PWR?
+L power:GND #PWR027
 U 1 1 5DFF8E35
 P 6500 6450
-F 0 "#PWR?" H 6500 6200 50  0001 C CNN
+F 0 "#PWR027" H 6500 6200 50  0001 C CNN
 F 1 "GND" V 6505 6322 50  0000 R CNN
 F 2 "" H 6500 6450 50  0001 C CNN
@@
 	6250 6450 6500 6450
 $Comp
-L power:GND #PWR?
+L power:GND #PWR024
 U 1 1 5DFFD120
 P 2400 1950
-F 0 "#PWR?" H 2400 1700 50  0001 C CNN
+F 0 "#PWR024" H 2400 1700 50  0001 C CNN
 F 1 "GND" V 2405 1822 50  0000 R CNN
 F 2 "" H 2400 1950 50  0001 C CNN
@@
 $EndComp
 $Comp
-L power:GND #PWR?
+L power:GND #PWR025
 U 1 1 5DFFD4A4
 P 4250 2650
-F 0 "#PWR?" H 4250 2400 50  0001 C CNN
+F 0 "#PWR025" H 4250 2400 50  0001 C CNN
 F 1 "GND" V 4255 2522 50  0000 R CNN
 F 2 "" H 4250 2650 50  0001 C CNN
