File: PowerInterface.sch (KiCad schematic (older format))
At the start: 1 part, among them U2 AD9364BBCZ

Commit message: add some pmic library
Parts:
- U2: symbol MedusaLIB:AD9364BBCZ -> MedusaSDR-rescue:AD9364BBCZ-MedusaLIB
Changed lines of the file:
@@
 EESchema Schematic File Version 4
-LIBS:MedusaSDR-cache
 EELAYER 30 0
 EELAYER END
 $Descr A3 16535 11693
 encoding utf-8
-Sheet 8 11
+Sheet 8 12
 Title ""
 Date ""
@@
 $EndDescr
 $Comp
-L MedusaLIB:AD9364BBCZ U2
+L MedusaSDR-rescue:AD9364BBCZ-MedusaLIB U2
 U 2 1 5DDB8309
 P 8350 5200
