File: SoC.sch (KiCad schematic (older format))
At the start: 0 parts

Commit message: crot
Connections:
- wire segments 1 -> 0
Changed lines of the file:
@@
 EESchema Schematic File Version 4
+LIBS:MedusaSDR-cache
 EELAYER 30 0
 EELAYER END
-$Descr A4 11693 8268
+$Descr A3 16535 11693
 encoding utf-8
-Sheet 2 2
-Title ""
-Date ""
-Rev ""
-Comp ""
-Comment1 ""
-Comment2 ""
-Comment3 ""
+Sheet 2 11
+Title "Some Interface"
+Date "2019-11-24"
+Rev "1"
+Comp "labseni"
+Comment1 "add some interface"
+Comment2 "change page set to A3"
+Comment3 "connect to fpga"
 Comment4 ""
 $EndDescr
-Wire Wire Line
-	2850 3150 2850 3650
+$Sheet
+S 4900 1200 1450 1200
+U 5DDDC62C
+F0 "PortB" 50
+F1 "PortB.sch" 50
+$EndSheet
+$Sheet
+S 1800 1100 1600 1150
+U 5DE660C3
+F0 "PortA" 50
+F1 "PortA.sch" 50
+$EndSheet
+$Sheet
+S 7450 1250 1350 1150
+U 5DEEA64B
+F0 "PortC" 50
+F1 "PortC.sch" 50
+$EndSheet
+$Sheet
+S 9600 1250 1600 1250
+U 5DF39D6D
+F0 "PortD" 50
+F1 "PortD.sch" 50
+$EndSheet
+$Sheet
+S 12150 1200 1300 1400
+U 5DF39DEE
+F0 "PortE" 50
+F1 "PortE.sch" 50
+$EndSheet
+$Sheet
+S 1900 3750 1650 1600
+U 5E03B0A5
+F0 "PowerPort" 50
+F1 "PowerPort.sch" 50
+$EndSheet
 $EndSCHEMATC
