File: SomeInterface.sch (KiCad schematic (older format))
At the start: 1 part, among them U2 AD9364BBCZ

Commit message: add some pmic library
Parts:
- U2: symbol MedusaLIB:AD9364BBCZ -> MedusaSDR-rescue:AD9364BBCZ-MedusaLIB
Changed lines of the file:
@@
 EESchema Schematic File Version 4
-LIBS:MedusaSDR-cache
 EELAYER 30 0
 EELAYER END
 $Descr A3 16535 11693
 encoding utf-8
-Sheet 7 11
+Sheet 7 12
 Title ""
 Date ""
@@
 	7400 8300 5000 8300
 $Comp
-L MedusaLIB:AD9364BBCZ U?
+L MedusaSDR-rescue:AD9364BBCZ-MedusaLIB U?
 U 1 1 5DDDB38D
 P 9700 5500
 AR Path="/5DE35227/5DDDB38D" Ref="U?"  Part="1"
 AR Path="/5DDAC124/5DDB81DD/5DDDB38D" Ref="U2"  Part="1"
+AR Path="/5DDDB38D" Ref="U2"  Part="1"
 F 0 "U2" H 9700 8293 60  0000 C CNN
 F 1 "AD9364BBCZ" H 9700 8187 60  0000 C CNN
